Commit message: multi rviz first test

File: src/lab357_james_bot/lab357_james_bot_description/urdf/neuronbot2.urdf (robot description, URDF)
Before this commit: robot lab357_james_bot_description, 6 links, 5 joints
Links:
- link base_link: geometry collision box size=0.25 0.25 0.25; visual mesh filename=package://lab357_james_bot_description/meshes/neuronbot2/ba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 scale=0.001 0.001 0.001
- link laser_frame: geometry collision mesh filename=package://lab357_james_bot_description/meshes/neuronbot2/la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 scale=0.001 0.001 0.001; visual mesh filename=package://lab357_james_bot_description/meshes/neuronbot2/la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 scale=0.001 0.001 0.001
- link wheel_left_link: geometry collision mesh filename=package://lab357_james_bot_description/meshes/neuronbot2/wh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 scale=0.001 0.001 0.001; visual mesh filename=package://lab357_james_bot_description/meshes/neuronbot2/wh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 scale=0.001 0.001 0.001
- link wheel_right_link: geometry collision mesh filename=package://lab357_james_bot_description/meshes/neuronbot2/wh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 scale=0.001 0.001 0.001; visual mesh filename=package://lab357_james_bot_description/meshes/neuronbot2/wh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 scale=0.001 0.001 0.001

File: src/lab357_james_bot/lab357_james_bot_description/urdf/neuronbot2_w_front_camera.urdf (robot description, URDF)
Before this commit: robot lab357_james_bot_description, 11 links, 10 joints
Links:
- link base_link: geometry collision box size=0.25 0.25 0.25; visual mesh filename=package://lab357_james_bot_description/meshes/neuronbot2/ba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 scale=0.001 0.001 0.001
- link laser_frame: geometry collision mesh filename=package://lab357_james_bot_description/meshes/neuronbot2/la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 scale=0.001 0.001 0.001; visual mesh filename=package://lab357_james_bot_description/meshes/neuronbot2/la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 scale=0.001 0.001 0.001
- link wheel_left_link: geometry collision mesh filename=package://lab357_james_bot_description/meshes/neuronbot2/wh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 scale=0.001 0.001 0.001; visual mesh filename=package://lab357_james_bot_description/meshes/neuronbot2/wh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 scale=0.001 0.001 0.001
- link wheel_right_link: geometry collision mesh filename=package://lab357_james_bot_description/meshes/neuronbot2/wh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 scale=0.001 0.001 0.001; visual mesh filename=package://lab357_james_bot_description/meshes/neuronbot2/wh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 scale=0.001 0.001 0.001

File: src/lab357_james_bot/lab357_james_bot_description/urdf/neuronbot2_w_top_camera.urdf (robot description, URDF)
Before this commit: robot lab357_james_bot_description, 11 links, 10 joints
Links:
- link base_link: geometry collision box size=0.25 0.25 0.25; visual mesh filename=package://lab357_james_bot_description/meshes/neuronbot2/ba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 scale=0.001 0.001 0.001
- link laser_frame: geometry collision mesh filename=package://lab357_james_bot_description/meshes/neuronbot2/la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 scale=0.001 0.001 0.001; visual mesh filename=package://lab357_james_bot_description/meshes/neuronbot2/la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 scale=0.001 0.001 0.001
- link wheel_left_link: geometry collision mesh filename=package://lab357_james_bot_description/meshes/neuronbot2/wh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 scale=0.001 0.001 0.001; visual mesh filename=package://lab357_james_bot_description/meshes/neuronbot2/wh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 scale=0.001 0.001 0.001
- link wheel_right_link: geometry collision mesh filename=package://lab357_james_bot_description/meshes/neuronbot2/wh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 scale=0.001 0.001 0.001; visual mesh filename=package://lab357_james_bot_description/meshes/neuronbot2/wh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 scale=0.001 0.001 0.001

File: src/lab357_james_bot/lab357_james_bot_description/urdf/turtlebot3_waffle.urdf (robot description, URDF)
Before this commit: robot turtlebot3_waffle, 13 links, 12 joints
Links:
- link base_link: geometry collision box size=0.266 0.266 0.094; visual mesh filename=package://lab357_james_bot_description/turtlebot3/meshes/ba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 scale=0.001 0.001 0.001
- link base_scan: geometry collision cylinder length=0.0315 radius=0.055; visual mesh filename=package://lab357_james_bot_description/turtlebot3/meshes/se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 scale=0.001 0.001 0.001
- link camera_link: geometry collision box size=0.012 0.132 0.020; visual mesh filename=package://lab357_james_bot_description/turtlebot3/meshes/se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
- link wheel_left_link: geometry collision cylinder length=0.018 radius=0.033; visual mesh filename=package://lab357_james_bot_description/turtlebot3/meshes/wh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 scale=0.001 0.001 0.001
- link wheel_right_link: geometry collision cylinder length=0.018 radius=0.033; visual mesh filename=package://lab357_james_bot_description/turtlebot3/meshes/wh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 scale=0.001 0.001 0.001
Joints:
- joint camera_depth_joint: origin xyz=0.005 0.028 0.013 rpy=-1.57 0 -1.57 -> xyz=0.005 0.028 0.013 rpy=0 0 0
- joint camera_depth_optical_joint: origin xyz=0 0 0 rpy=0 0 0 -> xyz=0 0 0 rpy=-1.57 0 -1.57
